Commit message: Fix: Controller bug fixed, spawn height updated. Drone flies successfully with 40N force.

File: src/hunter_drone_description/urdf/hunter.urdf.xacro (robot description, xacro)
@@ -3,7 +3,7 @@
     <xacro:property name="base_width" value="0.4"/>
     <xacro:property name="base_height" value="0.05"/>
-    <xacro:property name="rotor_radius" value="0.1"/>
+    <xacro:property name="base_mass" value="1.5"/> <xacro:property name="rotor_radius" value="0.1"/>
     <xacro:property name="rotor_height" value="0.02"/>
-    <material name="orange">
+    <xacro:property name="rotor_mass" value="0.05"/> <material name="orange">
         <color rgba="1.0 0.5 0.0 1.0"/>
     </material>
@@ -11,4 +11,20 @@
         <color rgba="0.0 0.0 0.0 1.0"/>
     </material>
+    <xacro:macro name="box_inertia" params="m w h d">
+        <inertial>
+            <mass value="${m}"/>
+            <inertia ixx="${(m/12) * (h*h + d*d)}" ixy="0.0" ixz="0.0"
+                     iyy="${(m/12) * (w*w + d*d)}" iyz="0.0"
+                     izz="${(m/12) * (w*w + h*h)}"/>
+        </inertial>
+    </xacro:macro>
+    <xacro:macro name="cylinder_inertia" params="m r h">
+        <inertial>
+            <mass value="${m}"/>
+            <inertia ixx="${(m/12) * (3*r*r + h*h)}" ixy="0.0" ixz="0.0"
+                     iyy="${(m/12) * (3*r*r + h*h)}" iyz="0.0"
+                     izz="${(m/2) * (r*r)}"/>
+        </inertial>
+    </xacro:macro>
     <link name="base_link">
         <visual>
@@ -23,5 +39,9 @@
             </geometry>
         </collision>
+        <xacro:box_inertia m="${base_mass}" w="${base_width}" h="${base_width}" d="${base_height}"/>
     </link>
+    <gazebo reference="base_link">
+        <material>Gazebo/Orange</material>
+    </gazebo>
     <xacro:macro name="rotor" params="prefix x y">
         <link name="${prefix}_rotor">
@@ -37,4 +57,5 @@
                 </geometry>
             </collision>
+            <xacro:cylinder_inertia m="${rotor_mass}" r="${rotor_radius}" h="${rotor_height}"/>
         </link>
         <joint name="${prefix}_joint" type="continuous">
@@ -44,4 +65,7 @@
             <axis xyz="0 0 1"/>
         </joint>
+        <gazebo reference="${prefix}_rotor">
+            <material>Gazebo/Black</material>
+        </gazebo>
     </xacro:macro>
     <xacro:rotor prefix="front_left" x="${base_width/2}" y="${base_width/2}"/>
@@ -49,3 +73,13 @@
     <xacro:rotor prefix="rear_left" x="-${base_width/2}" y="${base_width/2}"/>
     <xacro:rotor prefix="rear_right" x="-${base_width/2}" y="-${base_width/2}"/>
+    <gazebo>
+        <plugin name="gazebo_ros_force" filename="libgazebo_ros_force.so">
+            <ros>
+                <namespace>/hunter</namespace>
+                <remapping>gazebo_ros_force:=cmd_force</remapping>
+            </ros>
+            <link_name>base_link</link_name>
+            <force_frame>link</force_frame>
+        </plugin>
+    </gazebo>
 </robot>
